File: yellow_panda/clocks.kicad_sch (KiCad schematic)
At the start: 6 parts, among them Y1 8MHz, Y2 8MHz

Commit message: Everything is in place now
Swap STM MCU, Correct Switches,
add diodes, caps and resistors
Parts:
- C13, C14, C15, C16: value 22pF -> 15pF; footprint (none) -> Capacitor_SMD:C_0402_1005Metric_Pad0.74x0.62mm_HandSolder
- Y1, Y2: footprint (none) -> Crystal:Crystal_SMD_Abracon_ABM3B-4Pin_5.0x3.2mm
Changed lines of the file:
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@@
 (kicad_sch
-	(version 20231120)
+	(version 20250114)
 	(generator "eeschema")
-	(generator_version "8.0")
+	(generator_version "9.0")
 	(paper "A4")
 	(title_block
@@
 		(shape bidirectional)
 		(at 104.14 85.09 0)
-		(fields_autoplaced yes)
 		(effects
 			(font
@@
 		(shape bidirectional)
 		(at 74.93 85.09 180)
-		(fields_autoplaced yes)
 		(effects
 			(font
@@
 		(shape bidirectional)
 		(at 217.17 86.36 0)
-		(fields_autoplaced yes)
 		(effects
 			(font
@@
 		(shape bidirectional)
 		(at 187.96 86.36 180)
-		(fields_autoplaced yes)
 		(effects
 			(font
@@
 		(fields_autoplaced yes)
 		(property "Reference" "C16"
-			(at 217.17 92.71 0)
+			(at 217.17 92.7099 0)
 			(effects
 				(font
@@
 			)
 		)
-		(property "Value" "22pF"
-			(at 217.17 95.25 0)
+		(property "Value" "15pF"
+			(at 217.17 95.2499 0)
 			(effects
 				(font
@@
 			)
 		)
-		(property "Footprint" ""
+		(property "Footprint" "Capacitor_SMD:C_0402_1005Metric_Pad0.74x0.62mm_HandSolder"
 			(at 214.3252 97.79 0)
 			(effects
@@
 			)
 		)
-		(property "Footprint" ""
+		(property "Footprint" "Crystal:Crystal_SMD_Abracon_ABM3B-4Pin_5.0x3.2mm"
 			(at 88.9 85.09 0)
 			(effects
@@
 			)
 		)
-		(property "Value" "22pF"
+		(property "Value" "15pF"
 			(at 80.01 93.98 0)
 			(effects
@@
 			)
 		)
-		(property "Footprint" ""
+		(property "Footprint" "Capacitor_SMD:C_0402_1005Metric_Pad0.74x0.62mm_HandSolder"
 			(at 78.4352 96.52 0)
 			(effects
@@
 		(fields_autoplaced yes)
 		(property "Reference" "C14"
-			(at 104.14 91.44 0)
+			(at 104.14 91.4399 0)
 			(effects
 				(font
@@
 			)
 		)
-		(property "Value" "22pF"
-			(at 104.14 93.98 0)
+		(property "Value" "15pF"
+			(at 104.14 93.9799 0)
 			(effects
 				(font
@@
 			)
 		)
-		(property "Footprint" ""
+		(property "Footprint" "Capacitor_SMD:C_0402_1005Metric_Pad0.74x0.62mm_HandSolder"
 			(at 101.2952 96.52 0)
 			(effects
@@
 			)
 		)
-		(property "Value" "22pF"
+		(property "Value" "15pF"
 			(at 193.04 95.25 0)
 			(effects
@@
 			)
 		)
-		(property "Footprint" ""
+		(property "Footprint" "Capacitor_SMD:C_0402_1005Metric_Pad0.74x0.62mm_HandSolder"
 			(at 191.4652 97.79 0)
 			(effects
@@
 			)
 		)
-		(property "Footprint" ""
+		(property "Footprint" "Crystal:Crystal_SMD_Abracon_ABM3B-4Pin_5.0x3.2mm"
 			(at 201.93 86.36 0)
 			(effects
