File: yellow_panda/yellow_panda.kicad_pcb (KiCad board)
At the start: 2 copper layers, 306 x 132.4 mm, 212 parts, among them P1 USB_C_Plug_USB2.0, P2 USB_C_Plug_USB2.0, U1 STM32F103C8T6, U2 STM32F103C8T6, U3 LT1963AxST-3.3, U4 LT1963AxST-3.3

Commit message: Everything is in place now
Swap STM MCU, Correct Switches,
add diodes, caps and resistors
Parts:
- removed the D33 at (354.6, 147.1)
- removed the D34 at (354.6, 130.1)
- removed the D35 at (354.6, 113.1)
- removed the D36 at (354.6, 96.1)
- removed the D37 at (336.6, 147.1)
- removed the D38 at (336.6, 130.1)
- removed the D39 at (336.6, 113.1)
- removed the D40 at (336.6, 96.1)
- removed the D41 at (336.6, 79.1)
- removed the D42 at (318.6, 142.0)
- removed the D43 at (318.6, 125.0)
- removed the D44 at (318.6, 108.0)
- removed the D45 at (318.6, 91.0)
- removed the D46 at (318.6, 74.0)
- removed the D47 at (300.6, 136.9)
- removed the D48 at (300.6, 119.9)
- removed the D49 at (300.6, 102.9)
- removed the D50 at (300.6, 85.9)
- removed the D51 at (300.6, 68.9)
- removed the D52 at (282.6, 142.0)
- removed the D53 at (282.6, 125.0)
- removed the D54 at (282.6, 108.0)
- removed the D55 at (282.6, 91.0)
- removed the D56 at (282.6, 74.0)
- removed the D57 at (264.6, 147.1)
- removed the D58 at (264.6, 130.1)
- removed the D59 at (264.6, 113.1)
- removed the D60 at (264.6, 96.1)
- removed the D61 at (264.6, 79.1)
- removed the D62 at (646.5, 97.3)
- removed the D63 at (646.5, 100.6)
- removed the D64 at (646.5, 104.0)
- removed D71, D72, D73: ~, Diode_SMD:D_SOD-123
- removed S33, S34, S35, S36, S37, S38, S39, S40, S41, S42, S43, S44, S45, S46, S47, S48, S49, S50, S51, S52, S53, S54, S55, S56, S57, S58, S59, S60, S61, S62, S63, S64: , kiswitch/hotswaps:SW_Hotswap_Kailh_Choc_V1_Plated
- removed SW69, SW70, SW71, SW72, SW73: ~, kiswitch/hotswaps:SW_Hotswap_Kailh_Choc_V1_Plated_1.00u
- added ?: , clipboard:bf87ff4d-921f-4e46-abc4-457b704bfae1, F.Cu at (213.8, 167.6)
- added ?: , clipboard:bf87ff4d-921f-4e46-abc4-457b704bfae1, F.Cu at (188.8, 167.8)
- added C1: 10uF, Capacitor_SMD:C_1206_3216Metric_Pad1.33x1.80mm_HandSolder, B.Cu at (187.4, 112.8)
- added C10: 10uF, Capacitor_SMD:C_1206_3216Metric_Pad1.33x1.80mm_HandSolder, B.Cu at (183.6, 127.2)
- added C11: 15pF, Capacitor_SMD:C_0402_1005Metric_Pad0.74x0.62mm_HandSolder, B.Cu at (190.8, 138.0)
- added C12: 15pF, Capacitor_SMD:C_0402_1005Metric_Pad0.74x0.62mm_HandSolder, B.Cu at (189.4, 132.4)
- added C13: 10uF, Capacitor_SMD:C_1206_3216Metric_Pad1.33x1.80mm_HandSolder, B.Cu at (218.7, 142.8)
- added C14: 100nF, Capacitor_SMD:C_0201_0603Metric_Pad0.64x0.40mm_HandSolder, B.Cu at (220.5, 141.0)
- added C15: 100nF, Capacitor_SMD:C_0201_0603Metric_Pad0.64x0.40mm_HandSolder, B.Cu at (231.8, 128.2)
- added C16: 100nF, Capacitor_SMD:C_0201_0603Metric_Pad0.64x0.40mm_HandSolder, B.Cu at (231.8, 129.2)
- added C17: 100nF, Capacitor_SMD:C_0201_0603Metric_Pad0.64x0.40mm_HandSolder, B.Cu at (233.0, 140.0)
- added C18: 100nF, Capacitor_SMD:C_0201_0603Metric_Pad0.64x0.40mm_HandSolder, B.Cu at (233.0, 141.0)
- added C19: 15pF, Capacitor_SMD:C_0402_1005Metric_Pad0.74x0.62mm_HandSolder, B.Cu at (211.2, 132.4)
- added C2: 10uF, Capacitor_SMD:C_1206_3216Metric_Pad1.33x1.80mm_HandSolder, B.Cu at (187.4, 116.4)
- added C20: 15pF, Capacitor_SMD:C_0402_1005Metric_Pad0.74x0.62mm_HandSolder, B.Cu at (212.4, 138.0)
- added C21: 100nF, Capacitor_SMD:C_0201_0603Metric_Pad0.64x0.40mm_HandSolder, B.Cu at (182.8, 141.2)
- added C22: 100nF, Capacitor_SMD:C_0201_0603Metric_Pad0.64x0.40mm_HandSolder, B.Cu at (211.2, 130.6)
- added C3: 10uF, Capacitor_SMD:C_1206_3216Metric_Pad1.33x1.80mm_HandSolder, B.Cu at (218.6, 109.0)
- added C4: 10uF, Capacitor_SMD:C_1206_3216Metric_Pad1.33x1.80mm_HandSolder, B.Cu at (219.0, 119.6)
- added C5: 100nF, Capacitor_SMD:C_0201_0603Metric_Pad0.64x0.40mm_HandSolder, B.Cu at (170.4, 129.8)
- added C6: 100nF, Capacitor_SMD:C_0201_0603Metric_Pad0.64x0.40mm_HandSolder, B.Cu at (171.0, 128.8)
- added C7: 100nF, Capacitor_SMD:C_0201_0603Metric_Pad0.64x0.40mm_HandSolder, B.Cu at (182.4, 129.4)
- added C8: 100nF, Capacitor_SMD:C_0201_0603Metric_Pad0.64x0.40mm_HandSolder, B.Cu at (171.2, 141.4)
- added C9: 100nF, Capacitor_SMD:C_0201_0603Metric_Pad0.64x0.40mm_HandSolder, B.Cu at (171.2, 142.6)
- added D65: ~, Diode_SMD:D_SOD-123, B.Cu at (333.0, 177.4)
- added D66: ~, Diode_SMD:D_SOD-123, B.Cu at (351.0, 177.4)
- added D67: ~, Diode_SMD:D_SOD-123, B.Cu at (234.6, 206.6)
- added LCD1: I2C LCD, LCD:MODULE_358, F.Cu at (176.8, 135.5)
- added LCD2: I2C LCD, LCD:MODULE_358, F.Cu at (226.0, 135.0)
- added P3: Master Connection Plug, Custom Lib:USB_C_Receptacle_GCT_USB4110, F.Cu at (182.9, 181.2)
- added P4: Slave Connection Plug, Custom Lib:USB_C_Receptacle_GCT_USB4110, F.Cu at (219.6, 179.8)
- added R3: 10k, Resistor_SMD:R_0402_1005Metric_Pad0.72x0.64mm_HandSolder, B.Cu at (187.7, 169.1)
- added R4: 10k, Resistor_SMD:R_0402_1005Metric_Pad0.72x0.64mm_HandSolder, B.Cu at (214.6, 168.6)
- added SW65: SW_SPDT, Custom Lib:SLW-66527511-SMT-TR_CUD, F.Cu at (191.2, 170.6)
- added SW66: SW_SPDT, Custom Lib:SLW-66527511-SMT-TR_CUD, F.Cu at (211.4, 170.4)
- added SW67: SW_Push, Custom Lib:SW_TL3330_EWI, F.Cu at (170.6, 96.6)
- added Y1: 8MHz, Crystal:Crystal_SMD_Abracon_ABM3B-4Pin_5.0x3.2mm, B.Cu at (190.0, 135.2)
- added Y2: 8MHz, Crystal:Crystal_SMD_Abracon_ABM3B-4Pin_5.0x3.2mm, B.Cu at (212.0, 135.2)
- D1, D70: value ~ -> D_Schottky; footprint Diode_SMD:D_SOD-123 -> PCM_JLCPCB:D_SOT-23; moved to B.Cu
- D10, D11, D12, D13, D14, D15, D16, D17, D18, D19, D20, D21, D22, D23, D24, D25, D26, D27, D28, D29, D30, D31, D32, D33, D34, D35, D36, D37, D38, D39, D40, D41, D42, D43, D44, D45, D46, D47, D48, D49, D50, D51, D52, D53, D54, D55, D56, D57, D58, D59, D6, D60, D61, D62, D63, D64, D68, D69, D7, D8, D9, R1, R2: moved to B.Cu
- D2, D3, D4, D5: value ~ -> 5V; footprint Diode_SMD:D_SOD-123 -> PCM_JLCPCB:D_SOT-23; moved to B.Cu
- P1, P2: footprint usb-c:CONN16_USB4085-GF-A_GCT -> Custom Lib:USB_C_Receptacle_GCT_USB4110
- SW1, SW10, SW11, SW12, SW13, SW14, SW15, SW16, SW17, SW18, SW19, SW2, SW20, SW21, SW22, SW23, SW24, SW25, SW26, SW27, SW28, SW29, SW3, SW30, SW31, SW33, SW34, SW35, SW36, SW37, SW38, SW39, SW4, SW40, SW41, SW42, SW43, SW44, SW45, SW46, SW47, SW48, SW49, SW5, SW50, SW51, SW52, SW53, SW54, SW55, SW56, SW57, SW58, SW59, SW6, SW60, SW61, SW63, SW64, SW7, SW8, SW9: footprint kiswitch/hotswaps:SW_Hotswap_Kailh_Choc_V1_Plated_1.00u -> PCM_Switch_Keyboard_Hotswap_Kailh:SW_Hotswap_Kailh_Choc_V1_Plated_1.00u
- SW32, SW62: footprint kiswitch/hotswaps:SW_Hotswap_Kailh_Choc_V1_Plated_1.00u -> PCM_Switch_Keyboard_Hotswap_Kailh:SW_Hotswap_Kailh_Choc_V1_Plated_1.50u
- SW68: value ~ -> SW_Push; footprint kiswitch/hotswaps:SW_Hotswap_Kailh_Choc_V1_Plated_1.00u -> Custom Lib:SW_TL3330_EWI
- U1, U2: value STM32F103C8T6 -> LT1963AxST-3.3; footprint STM32F10:LQFP48_STM -> Package_TO_SOT_SMD:SOT-223-3_TabPin2
- U3, U4: value LT1963AxST-3.3 -> STM32F446RCTx; footprint Package_TO_SOT_SMD:SOT-223-3_TabPin2 -> Package_QFP:LQFP-64_10x10mm_P0.5mm
- moved D35 513.1 mm to (128.3, 199.0)
- moved D33 500.6 mm to (137.0, 172.4)
- moved D36 490.3 mm to (151.6, 202.2), turned to -10 degrees
- moved D34 483.1 mm to (155.1, 177.4)
- moved D37 467.7 mm to (172.4, 195.2), turned to 70 degrees
- moved D70 437.1 mm to (220.0, 179.6), turned to -60 degrees
- moved D55 386.6 mm to (261.0, 160.4)
- moved D68 386.3 mm to (264.8, 199.8), turned to 10 degrees
- moved D61 386.1 mm to (261.0, 177.4)
- moved SW62 385.4 mm to (235.0, 200.7), turned to -70 degrees
- moved D69 377.1 mm to (288.0, 197.8)
- moved D43 376.7 mm to (261.0, 126.6)
- moved D49 376.1 mm to (261.2, 143.4)
- moved SW68 371.4 mm to (233.8, 96.4), turned to -173 degrees
- moved D38 368.3 mm to (261.0, 109.6)
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Connections:
- D1 pad 1: /MasterSwitchMatrix/ROW0a -> +3.3V
- D10 pad 1: /MasterSwitchMatrix/ROW1a -> /MasterSwitchMatrix/ROW0a
- D12 pad 1: /MasterSwitchMatrix/ROW2a -> /MasterSwitchMatrix/ROW1a
- D13 pad 1: /MasterSwitchMatrix/ROW2a -> /MasterSwitchMatrix/ROW1a
- D14 pad 1: /MasterSwitchMatrix/ROW2a -> /MasterSwitchMatrix/ROW1a
- D15 pad 1: /MasterSwitchMatrix/ROW2a -> /MasterSwitchMatrix/ROW1a
- D16 pad 1: /MasterSwitchMatrix/ROW2a -> /MasterSwitchMatrix/ROW1a
- D18 pad 1: /MasterSwitchMatrix/ROW3a -> /MasterSwitchMatrix/ROW2a
- D19 pad 1: /MasterSwitchMatrix/ROW3a -> /MasterSwitchMatrix/ROW2a
- D2 pad 1: /MasterSwitchMatrix/ROW0a -> GND
- D2 pad 2: Net-(D2-A) -> /USB_D+a
- D20 pad 1: /MasterSwitchMatrix/ROW3a -> /MasterSwitchMatrix/ROW2a
- D21 pad 1: /MasterSwitchMatrix/ROW3a -> /MasterSwitchMatrix/ROW2a
- D22 pad 1: /MasterSwitchMatrix/ROW3a -> /MasterSwitchMatrix/ROW2a
- D24 pad 1: /MasterSwitchMatrix/ROW4a -> /MasterSwitchMatrix/ROW3a
- D25 pad 1: /MasterSwitchMatrix/ROW4a -> /MasterSwitchMatrix/ROW3a
- D26 pad 1: /MasterSwitchMatrix/ROW4a -> /MasterSwitchMatrix/ROW3a
- D27 pad 1: /MasterSwitchMatrix/ROW4a -> /MasterSwitchMatrix/ROW3a
- D28 pad 1: /MasterSwitchMatrix/ROW4a -> /MasterSwitchMatrix/ROW3a
- D3 pad 1: /MasterSwitchMatrix/ROW0a -> GND
- D3 pad 2: Net-(D3-A) -> /USB_D+b
- D30 pad 1: /MasterSwitchMatrix/ROW6a -> /MasterSwitchMatrix/ROW4a
- D31 pad 1: /MasterSwitchMatrix/ROW6a -> /MasterSwitchMatrix/ROW4a
- D32 pad 1: /MasterSwitchMatrix/ROW6a -> /MasterSwitchMatrix/ROW4a
- D33 pad 1: /SlaveSwitchMatrix/ROW0b -> /MasterSwitchMatrix/ROW4a
- D34 pad 1: /SlaveSwitchMatrix/ROW0b -> /MasterSwitchMatrix/ROW4a
- D35 pad 1: /SlaveSwitchMatrix/ROW0b -> /MasterSwitchMatrix/ROW6a
- D36 pad 1: /SlaveSwitchMatrix/ROW0b -> /MasterSwitchMatrix/ROW6a
- D37 pad 1: /SlaveSwitchMatrix/ROW0b -> /MasterSwitchMatrix/ROW6a
- D38 pad 1: /SlaveSwitchMatrix/ROW1b -> /SlaveSwitchMatrix/ROW0b
- D39 pad 1: /SlaveSwitchMatrix/ROW1b -> /SlaveSwitchMatrix/ROW0b
- D4 pad 1: /MasterSwitchMatrix/ROW0a -> GND
- D4 pad 2: Net-(D4-A) -> /USB_D-a
- D40 pad 1: /SlaveSwitchMatrix/ROW1b -> /SlaveSwitchMatrix/ROW0b
- D41 pad 1: /SlaveSwitchMatrix/ROW1b -> /SlaveSwitchMatrix/ROW0b
- D42 pad 1: /SlaveSwitchMatrix/ROW1b -> /SlaveSwitchMatrix/ROW0b
- D44 pad 1: /SlaveSwitchMatrix/ROW2b -> /SlaveSwitchMatrix/ROW1b
- D45 pad 1: /SlaveSwitchMatrix/ROW2b -> /SlaveSwitchMatrix/ROW1b
- D46 pad 1: /SlaveSwitchMatrix/ROW2b -> /SlaveSwitchMatrix/ROW1b
- D47 pad 1: /SlaveSwitchMatrix/ROW2b -> /SlaveSwitchMatrix/ROW1b
- D48 pad 1: /SlaveSwitchMatrix/ROW2b -> /SlaveSwitchMatrix/ROW1b
- D5 pad 1: /MasterSwitchMatrix/ROW0a -> GND
- D5 pad 2: Net-(D5-A) -> /USB_D-b
- D50 pad 1: /SlaveSwitchMatrix/ROW3b -> /SlaveSwitchMatrix/ROW2b
- D51 pad 1: /SlaveSwitchMatrix/ROW3b -> /SlaveSwitchMatrix/ROW2b
- D52 pad 1: /SlaveSwitchMatrix/ROW3b -> /SlaveSwitchMatrix/ROW2b
- D53 pad 1: /SlaveSwitchMatrix/ROW3b -> /SlaveSwitchMatrix/ROW2b
- D54 pad 1: /SlaveSwitchMatrix/ROW3b -> /SlaveSwitchMatrix/ROW2b
- D56 pad 1: /SlaveSwitchMatrix/ROW4b -> /SlaveSwitchMatrix/ROW3b
- D57 pad 1: /SlaveSwitchMatrix/ROW4b -> /SlaveSwitchMatrix/ROW3b
- D58 pad 1: /SlaveSwitchMatrix/ROW4b -> /SlaveSwitchMatrix/ROW3b
- D59 pad 1: /SlaveSwitchMatrix/ROW4b -> /SlaveSwitchMatrix/ROW3b
- D6 pad 1: /MasterSwitchMatrix/ROW1a -> /MasterSwitchMatrix/ROW0a
- D60 pad 1: /SlaveSwitchMatrix/ROW4b -> /SlaveSwitchMatrix/ROW3b
- D62 pad 1: /SlaveSwitchMatrix/ROW6b -> /SlaveSwitchMatrix/ROW4b
- D63 pad 1: /SlaveSwitchMatrix/ROW6b -> /SlaveSwitchMatrix/ROW4b
- D64 pad 1: /SlaveSwitchMatrix/ROW6b -> /SlaveSwitchMatrix/ROW4b
- D68 pad 1: /SlaveSwitchMatrix/ROW5b -> /SlaveSwitchMatrix/ROW6b
- D69 pad 1: /SlaveSwitchMatrix/ROW5b -> /SlaveSwitchMatrix/ROW6b
- D7 pad 1: /MasterSwitchMatrix/ROW1a -> /MasterSwitchMatrix/ROW0a
- D70 pad 1: /SlaveSwitchMatrix/ROW5b -> +3.3V
- D8 pad 1: /MasterSwitchMatrix/ROW1a -> /MasterSwitchMatrix/ROW0a
- D9 pad 1: /MasterSwitchMatrix/ROW1a -> /MasterSwitchMatrix/ROW0a
- R1 pad 1: GNDR -> GND
- R2 pad 1: GNDR -> GND
- SW1 pad 2: Net-(D1-A) -> Net-(D6-A)
- SW10 pad 2: Net-(D10-A) -> Net-(D15-A)
- SW11 pad 2: Net-(D11-A) -> Net-(D16-A)
- SW12 pad 2: Net-(D12-A) -> Net-(D17-A)
- SW13 pad 2: Net-(D13-A) -> Net-(D18-A)
- SW14 pad 2: Net-(D14-A) -> Net-(D19-A)
- SW15 pad 2: Net-(D15-A) -> Net-(D20-A)
- SW16 pad 2: Net-(D16-A) -> Net-(D21-A)
- SW17 pad 2: Net-(D17-A) -> Net-(D22-A)
- SW18 pad 2: Net-(D18-A) -> Net-(D23-A)
- SW19 pad 2: Net-(D19-A) -> Net-(D24-A)
- SW2 pad 2: Net-(D2-A) -> Net-(D7-A)
- SW20 pad 2: Net-(D20-A) -> Net-(D25-A)
- SW21 pad 2: Net-(D21-A) -> Net-(D26-A)
- SW22 pad 2: Net-(D22-A) -> Net-(D27-A)
- SW23 pad 2: Net-(D23-A) -> Net-(D28-A)
- SW24 pad 2: Net-(D24-A) -> Net-(D29-A)
- SW25 pad 2: Net-(D25-A) -> Net-(D30-A)
- SW26 pad 2: Net-(D26-A) -> Net-(D31-A)
- SW27 pad 2: Net-(D27-A) -> Net-(D32-A)
- SW28 pad 2: Net-(D28-A) -> Net-(D33-A)
- SW29 pad 2: Net-(D29-A) -> Net-(D34-A)
- SW3 pad 2: Net-(D3-A) -> Net-(D8-A)
- SW30 pad 2: Net-(D30-A) -> Net-(D35-A)
- SW31 pad 2: Net-(D31-A) -> Net-(D36-A)
- SW32 pad 2: Net-(D32-A) -> Net-(D37-A)
- SW33 pad 1: /SlaveSwitchMatrix/COL1b -> /SlaveSwitchMatrix/COL0b
- SW33 pad 2: Net-(D33-A) -> Net-(D38-A)
- SW34 pad 1: /SlaveSwitchMatrix/COL2b -> /SlaveSwitchMatrix/COL1b
- SW34 pad 2: Net-(D34-A) -> Net-(D39-A)
- SW35 pad 1: /SlaveSwitchMatrix/COL3b -> /SlaveSwitchMatrix/COL2b
- SW35 pad 2: Net-(D35-A) -> Net-(D40-A)
- SW36 pad 1: /SlaveSwitchMatrix/COL4b -> /SlaveSwitchMatrix/COL3b
- SW36 pad 2: Net-(D36-A) -> Net-(D41-A)
- SW37 pad 1: /SlaveSwitchMatrix/COL5b -> /SlaveSwitchMatrix/COL4b
- SW37 pad 2: Net-(D37-A) -> Net-(D42-A)
- SW38 pad 2: Net-(D38-A) -> Net-(D43-A)
- SW39 pad 2: Net-(D39-A) -> Net-(D44-A)
- SW4 pad 2: Net-(D4-A) -> Net-(D9-A)
- SW40 pad 2: Net-(D40-A) -> Net-(D45-A)
- SW41 pad 2: Net-(D41-A) -> Net-(D46-A)
- SW42 pad 2: Net-(D42-A) -> Net-(D47-A)
- SW43 pad 2: Net-(D43-A) -> Net-(D48-A)
- SW44 pad 2: Net-(D44-A) -> Net-(D49-A)
- SW45 pad 2: Net-(D45-A) -> Net-(D50-A)
- SW46 pad 2: Net-(D46-A) -> Net-(D51-A)
- SW47 pad 2: Net-(D47-A) -> Net-(D52-A)
- SW48 pad 2: Net-(D48-A) -> Net-(D53-A)
- SW49 pad 2: Net-(D49-A) -> Net-(D54-A)
- SW5 pad 2: Net-(D5-A) -> Net-(D10-A)
- SW50 pad 2: Net-(D50-A) -> Net-(D55-A)
- SW51 pad 2: Net-(D51-A) -> Net-(D56-A)
- SW52 pad 2: Net-(D52-A) -> Net-(D57-A)
- SW53 pad 2: Net-(D53-A) -> Net-(D58-A)
- SW54 pad 2: Net-(D54-A) -> Net-(D59-A)
- SW55 pad 2: Net-(D55-A) -> Net-(D60-A)
- SW56 pad 2: Net-(D56-A) -> Net-(D61-A)
- SW57 pad 2: Net-(D57-A) -> Net-(D62-A)
- SW58 pad 2: Net-(D58-A) -> Net-(D63-A)
- SW59 pad 2: Net-(D59-A) -> Net-(D64-A)
- SW6 pad 2: Net-(D6-A) -> Net-(D11-A)
- SW60 pad 2: Net-(D60-A) -> Net-(D65-A)
- SW61 pad 2: Net-(D61-A) -> Net-(D66-A)
- SW62 pad 1: /SlaveSwitchMatrix/COL3b -> /SlaveSwitchMatrix/COL0b
- SW62 pad 2: Net-(D62-A) -> Net-(D67-A)
- SW63 pad 1: /SlaveSwitchMatrix/COL4b -> /SlaveSwitchMatrix/COL1b
- SW63 pad 2: Net-(D63-A) -> Net-(D68-A)
- SW64 pad 1: /SlaveSwitchMatrix/COL5b -> /SlaveSwitchMatrix/COL2b
- SW64 pad 2: Net-(D64-A) -> Net-(D69-A)
- SW68 pad 1: /SlaveSwitchMatrix/COL0b -> /STM MCUs/RESETb
- SW68 pad 2: Net-(D68-A) -> GND
- SW7 pad 2: Net-(D7-A) -> Net-(D12-A)
- SW8 pad 2: Net-(D8-A) -> Net-(D13-A)
- SW9 pad 2: Net-(D9-A) -> Net-(D14-A)
- U1 pad 1: Net-(U1B-VBAT) -> +5V
- U1 pad 2: unconnected-(U1A-PC13-Pad2) -> GND
- U1 pad 3: unconnected-(U1A-PC14-OSC32_IN-Pad3) -> +3.3V
- U2 pad 1: Net-(U2B-VBAT) -> +5V
- U2 pad 2: unconnected-(U2A-PC13-Pad2) -> GND
- U2 pad 3: unconnected-(U2A-PC14-OSC32_IN-Pad3) -> Net-(D1-A)
- U3 pad 1: +5V -> +3.3V
- U3 pad 2: GND -> unconnected-(U3-PC13-Pad2)
- U3 pad 3: +3.3V -> unconnected-(U3-PC14-Pad3)
- U4 pad 1: +5V -> +3.3V
- U4 pad 2: GND -> unconnected-(U4-PC13-Pad2)
- U4 pad 3: +3.3V -> unconnected-(U4-PC14-Pad3)
Other:
- board size 306 x 132.4 mm -> 305.9 x 130.6 mm
- board text added: "Computer"
- board text added: "Flash Mode"
- board text added: "Reset"
- board text added: "Split Connector"

Commit message: Added some routing to power lines
Parts:
- moved C11 13.5 mm to (182.8, 148.8)
- moved Y1 13.5 mm to (182.0, 146.0)
- moved C12 13.5 mm to (181.4, 143.2)
- moved C1 11.9 mm to (192.6, 123.6), turned to -90 degrees
- moved U1 8.77 mm to (188.0, 116.5), turned to 90 degrees
- moved C2 6.10 mm to (187.5, 122.5)
- moved D4 5.17 mm to (177.8, 104.5), turned to -100 degrees
- moved D2 3.21 mm to (177.5, 100.5), turned to 170 degrees
- moved C5 0.83 mm to (170.0, 130.5)
- moved R1 0.58 mm to (188.5, 102.5)
- moved C6 0.57 mm to (170.5, 129.0), turned to 90 degrees
Connections:
- net /USB_D+a renamed /USB_Da+
- net /USB_D+b renamed /USB_Db+
- net /USB_D-a renamed /USB_Da-
- net /USB_D-b renamed /USB_Db-
- P1 pad A1: GNDR -> GND
- P1 pad A12: GNDR -> GND
- P1 pad B1: GNDR -> GND
- P1 pad B12: GNDR -> GND
- P1 pad S1: GNDR -> GND
- P2 pad A1: GNDR -> GND
- P2 pad A12: GNDR -> GND
- P2 pad B1: GNDR -> GND
- P2 pad B12: GNDR -> GND
- P2 pad S1: GNDR -> GND
Routing:
- net +3.3V: track 0.00 -> 143.7 mm, vias 0 -> 2
- net GND: track 0.00 -> 63.6 mm, vias 0 -> 19
- net +5V: track 0.00 -> 45.7 mm, vias 0 -> 4
- net /USB_Da-: track 0.00 -> 10.8 mm, vias 0 -> 1
- net /USB_Da+: track 0.00 -> 9.57 mm, vias 0 -> 1
- net /STM MCUs/RESETa: track 0.00 -> 8.74 mm
- net /STM MCUs/SW_BOOT0a: track 0.00 -> 2.04 mm, vias 0 -> 1
- net /STM MCUs/OSC OUTa: track 0.00 -> 1.94 mm
- net /STM MCUs/OSC INa: track 0.00 -> 1.86 mm
- net Net-(P1-CC): track 0.00 -> 0.98 mm, vias 0 -> 1
- added copper zone on B.Cu, net GND
