File: yellow_panda/i2c_devices.kicad_sc.kicad_sch (KiCad schematic)
At the start: 5 parts, among them P3 Master Connection Plug, P4 Slave Connection Plug

Commit message: rev0.1a - master half done
Parts:
- removed LCD1, LCD2: I2C LCD, LCD:MODULE_358, symbol Interface_Expansion:PCF8574
- added U7, U8: 358, LCD:MODULE_358, symbol led:358
- renumbered D70 to D5
Connections:
- net +3.3V: now also U7.9 (VCC)
- net GND: now also U7.10 (GND)
- new net CSa: U7.5 (TFT_CS)
- new net DataCommanda: U7.7 (D/C)
- new net LCDReseta: U7.8 (RESET)
- new net MISOa: U7.2 (MISO)
- new net MOSIa: U7.4 (MOSI)
- new net SCKa: U7.3 (SCK)
- new net SDCSa: U7.6 (CARD_CS)
- new net ScreenBrighta: U7.1 (LITE)
- no-connect marks 28 -> 4
