File: yellow_panda/devices.kicad_sc.kicad_sch (KiCad schematic)
At the start: 7 parts, among them J1 Conn_ST_STDC14, J2 Conn_ST_STDC14, P3 Master Connection Plug, P4 Slave Connection Plug, U7 358, U8 358

Commit message: Finished the design
Parts:
- removed D4: D_Schottky, PCM_JLCPCB:D_SOT-23, symbol Device:D_Schottky
Connections:
- net +3.3V: now also J1.3 (VCC), U8.9 (VCC); no longer P3.A4 (VBUS), P3.A9 (VBUS), P3.B4 (VBUS), P3.B9 (VBUS)
- net GND: now also J1.5 (GND), J1.7 (GND), U8.10 (GND)
- net RESETb: now reaches J1.12 (~{RST})
- net UART_RXb: now reaches J1.13 (VCP_RX)
- net UART_TXb: now reaches J1.14 (VCP_TX)
- net SWDIOb: now reaches J1.4 (JTMS/SWDIO)
- net SWCLKb: now reaches J1.6 (JCLK/SWCLK)
- net SWOb: now reaches J1.8 (JTDO/SWO)
- net ScreenBrightb: now reaches U8.1 (LITE)
- net MISOb: now reaches U8.2 (MISO)
- net SCKb: now reaches U8.3 (SCK)
- net MOSIb: now reaches U8.4 (MOSI)
- net CSb: now reaches U8.5 (TFT_CS)
- net SDCSb: now reaches U8.6 (CARD_CS)
- net DataCommandb: now reaches U8.7 (D/C)
- net LCDResetb: now reaches U8.8 (RESET)
- net VBUS MASTER HALF: now reaches P4.A4 (VBUS), P4.A9 (VBUS), P4.B4 (VBUS), P4.B9 (VBUS)
- net SDLb renamed SCLb
- new net +5V: P3.A4 (VBUS), P3.A9 (VBUS), P3.B4 (VBUS), P3.B9 (VBUS)
Other:
- moved on the sheet: U8

Commit message: v0.1b
Parts:
- removed P3: Master Connection Plug, Custom Lib:USB_C_Receptacle_GCT_USB4110, symbol Connector:USB_C_Plug_USB2.0
- removed P4: Slave Connection Plug, Custom Lib:USB_C_Receptacle_GCT_USB4110, symbol Connector:USB_C_Plug_USB2.0
- added USBC3, USBC4: TYPE-C-31-M-12, easyeda2kicad:USB-C_SMD-TYPE-C-31-M-12_1, symbol easyeda2kicad:TYPE-C-31-M-12
- J1, J2, U7, U8: now not fitted
Connections:
- net +5V: now also USBC3.A4B9 (VBUS), USBC3.B4A9 (VBUS)
- net GND: now also USBC3.1 (EH), USBC3.2 (EH), USBC3.3 (EH), USBC3.4 (EH), USBC3.A1B12 (GND), USBC3.B1A12 (GND), USBC4.1 (EH), USBC4.2 (EH), USBC4.3 (EH), USBC4.4 (EH), USBC4.A1B12 (GND), USBC4.B1A12 (GND)
- net SCLa: now also USBC3.A6 (DP1), USBC3.B6 (DP2)
- net SCLb: now also USBC4.A6 (DP1), USBC4.B6 (DP2)
- net SDAa: now also USBC3.A7 (DN1), USBC3.B7 (DN2)
- net SDAb: now also USBC4.A7 (DN1), USBC4.B7 (DN2)
- net VBUS MASTER HALF: now also USBC4.A4B9 (VBUS), USBC4.B4A9 (VBUS)
- no-connect marks 4 -> 8
