File: pandakbd/devices.kicad_sc.kicad_sch (KiCad schematic)
At the start: 6 parts, among them J1 Conn_ST_STDC14, J2 Conn_ST_STDC14, U7 358, U8 358

Commit message: rev2
Parts:
- removed J1, J2: Conn_ST_STDC14, Connector_PinHeader_1.27mm:PinHeader_2x07_P1.27mm_Horizontal, symbol Connector:Conn_ST_STDC14
- removed U7, U8: 358, LCD:MODULE_358, symbol led:358
- removed USBC3, USBC4: TYPE-C-31-M-12, easyeda2kicad:USB-C_SMD-TYPE-C-31-M-12_1, symbol easyeda2kicad:TYPE-C-31-M-12
Connections:
- no-connect marks 8 -> 0
