File: pandakbd/master_matrix.kicad_sch (KiCad schematic)
At the start: 64 parts, among them SW1 1N4148W, SW10 1N4148W, SW11 1N4148W, SW12 1N4148W, SW13 1N4148W, SW14 1N4148W, SW15 1N4148W, SW16 1N4148W, SW17 1N4148W, SW18 1N4148W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

Commit message: rev2
Parts:
- renumbered D6 to D1, D15 to D10, D16 to D11, D17 to D12, D18 to D13, D19 to D14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
Other:
- moved on the sheet: D1, D10, D11, D12, D13, D14, D15, D16, D17, D18, D19, D2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
