File: pandakbd/powerleds.kicad_sch (KiCad schematic)
At the start: 8 parts

Commit message: rev2
Parts:
- removed D5: GLED, easyeda2kicad:LED0805-R-RD, symbol Device:LED
- removed D70: YLED, easyeda2kicad:LED0805-R-RD, symbol Device:LED
- removed R11: 33Ω, Resistor_SMD:R_0603_1608Metric, symbol Device:R
- removed R12: 300, Resistor_SMD:R_0603_1608Metric, symbol Device:R
