File: pandakbd/slave_matrix.kicad_sch (KiCad schematic)
At the start: 64 parts, among them SW33 1N4148W, SW34 1N4148W, SW35 1N4148W, SW36 1N4148W, SW37 1N4148W, SW38 1N4148W, SW39 1N4148W, SW40 1N4148W, SW41 1N4148W, SW42 1N4148W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

Commit message: rev2
Parts:
- renumbered D38 to D33, D39 to D34, D40 to D35, D41 to D36, D42 to D37, D43 to D38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
Other:
- moved on the sheet: D33, D34, D35, D36, D37, D38, D39, D40, D41, D42, D43, D44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
