File: pandakbd/right.kicad_sch (KiCad schematic)
At the start: 34 parts, among them J2 Conn_ST_STDC14, SW66 MK-12C03-G015, U10 GT-TC020A-H035-L05, U6 LDI1117, U7 USBLC6-2SC6_C5261088, U8 358, U9 STM32F446RCTx, Y2 8MHz

Commit message: prepare placing components
Parts:
- U7: footprint easyeda2kicad:SOT-23-6_L2.9-W1.6-P0.95-LS2.8-BR -> Package_TO_SOT_SMD:SOT-23-6
Changed lines of the file:
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@@
 			)
 		)
-		(property "Footprint" "easyeda2kicad:SOT-23-6_L2.9-W1.6-P0.95-LS2.8-BR"
+		(property "Footprint" "Package_TO_SOT_SMD:SOT-23-6"
 			(at 85.09 60.96 0)
 			(effects
