File: pcbs/rev2.0/migrane.kicad_pcb (KiCad board)
At the start: 2 copper layers, 308.1 x 146 mm, 334 parts, among them J1 Conn_ST_STDC14, J2 Conn_ST_STDC14, SW1 1N4148W, SW10 1N4148W, SW11 1N4148W, SW12 1N4148W, SW13 1N4148W, SW14 1N4148W, SW15 1N4148W, SW16 1N4148W, SW17 1N4148W, SW18 1N4148W, SW19 1N4148W, SW2 1N4148W, SW20 1N4148W, SW21 1N4148W, SW22 1N4148W, SW23 1N4148W, SW24 1N4148W, SW25 1N4148W, SW26 1N4148W, SW27 1N4148W, SW28 1N4148W, SW29 1N4148W, SW3 1N4148W, SW30 1N4148W, SW31 1N4148W, SW32 1N4148W, SW33 1N4148W, SW34 1N4148W, SW35 1N4148W, SW36 1N4148W, SW37 1N4148W, SW38 1N4148W, SW39 1N4148W, SW4 1N4148W, SW40 1N4148W, SW41 1N4148W, SW42 1N4148W, SW43 1N4148W, SW44 1N4148W, SW45 1N4148W, SW46 1N4148W, SW47 1N4148W, SW48 1N4148W, SW49 1N4148W, SW5 1N4148W, SW50 1N4148W, SW51 1N4148W, SW52 1N4148W, SW53 1N4148W, SW54 1N4148W, SW55 1N4148W, SW56 1N4148W, SW57 1N4148W, SW58 1N4148W, SW59 1N4148W, SW6 1N4148W, SW60 1N4148W, SW61 1N4148W, SW62 1N4148W, SW63 1N4148W, SW64 1N4148W, SW65 MK-12C03-G015, SW69 MK-12C03-G015, SW7 1N4148W, SW8 1N4148W, SW9 1N4148W, U1 LDI1117, U10 GT-TC020A-H035-L05, U11 GT-TC020A-H035-L05, U2 USBLC6-2SC6_C5261088, U3 358, U4 STM32F446RCTx, U5 GT-TC020A-H035-L05, U6 LDI1117, U7 USBLC6-2SC6_C5261088, U9 STM32F446RCTx, Y1 8MHz, Y2 8MHz

Commit message: start with leds
Parts:
- added LED23: SK6812mini-e, easyeda2kicad:LED-SMD_L3.2-W2.8-LS5.9_SK6812MINI-E, F.Cu at (-17.8, 60.2)
- added LED6: 4960, easyeda2kicad:LED-SMD_L3.2-W2.8-LS5.9_SK6812MINI-E, F.Cu at (-16.3, 48.5)
- added LED7: SK6812mini-e, easyeda2kicad:LED-SMD_L3.2-W2.8-LS5.9_SK6812MINI-E, F.Cu at (-16.3, 52.8)
- added SW66: MK-12C03-G015, easyeda2kicad:SW-SMD_MK-12C03-G015, F.Cu at (67.0, 47.6)
- added U8: 358, easyeda2kicad:MODULE_358, F.Cu at (92.1, 26.9)
- LED18: renamed from LED12; value 4960 -> SK6812mini-e
- LED7: renamed from LED6; value 4960 -> SK6812mini-e
- LED9: renamed from LED8; value SK6812mini-e -> 4960
- moved D9 1.47 mm to (120.5, 116.5)
- moved D8 0.76 mm to (101.5, 122.0)
- moved D7 0.61 mm to (83.5, 127.0)
- moved LED24 0.52 mm to (148.5, 163.2)
- moved D6 0.50 mm to (65.0, 126.5)
- moved LED18 0.43 mm to (148.5, 146.3)
- moved LED7 0.33 mm to (58.5, 129.3)
- moved LED9 0.30 mm to (94.5, 124.3)
- moved LED18 0.26 mm to (58.4, 163.3)
- moved LED20 0.26 mm to (94.7, 158.2)
- moved LED12 0.25 mm to (148.2, 129.3)
- moved LED8 0.16 mm to (76.5, 129.3)
- moved LED11 0.10 mm to (130.4, 124.1)
- moved LED19 0.10 mm to (76.4, 163.3)
- renumbered LED5 to LED1, LED9 to LED10, LED10 to LED11, LED11 to LED12, LED17 to LED13, LED16 to LED14, LED14 to LED16, LED13 to LED17, LED4 to LED2, LED23 to LED24, LED2 to LED4, LED1 to LED5, LED7 to LED8
Connections:
- LED1 pad 2: Net-(LED5-DOUT) -> Net-(LED1-DOUT)
- LED1 pad 4: Net-(LED4-DOUT) -> LEDs^{a}
- LED12 pad 4: Net-(LED11-DIN) (its old number) -> Net-(LED12-DIN)
- LED13 pad 2: Net-(LED17-DOUT) -> Net-(LED13-DOUT)
- LED13 pad 4: Net-(LED16-DOUT) -> Net-(LED13-DIN)
- LED14 pad 2: Net-(LED16-DOUT) -> Net-(LED14-DOUT)
- LED14 pad 4: Net-(LED15-DOUT) -> Net-(LED13-DOUT)
- LED16 pad 2: Net-(LED14-DOUT) -> Net-(LED16-DOUT)
- LED16 pad 4: Net-(LED13-DOUT) -> Net-(LED15-DOUT)
- LED17 pad 2: Net-(LED13-DOUT) -> Net-(LED17-DOUT)
- LED17 pad 4: Net-(LED13-DIN) -> Net-(LED16-DOUT)
- LED18 pad 2: Net-(LED11-DIN) (its old number) -> Net-(LED18-DOUT)
- LED18 pad 4: Net-(LED12-DIN) -> Net-(LED17-DOUT)
- LED2 pad 2: Net-(LED4-DOUT) -> Net-(LED2-DOUT)
- LED2 pad 4: Net-(LED3-DOUT) -> Net-(LED1-DOUT)
- LED24 pad 2: Net-(LED22-DIN) -> Net-(LED23-DIN)
- LED24 pad 4: Net-(LED23-DIN) -> Net-(LED18-DOUT)
- LED4 pad 2: Net-(LED2-DOUT) -> Net-(LED4-DOUT)
- LED4 pad 4: Net-(LED1-DOUT) -> Net-(LED3-DOUT)
- LED5 pad 2: Net-(LED1-DOUT) -> Net-(LED5-DOUT)
- LED5 pad 4: LEDsa -> Net-(LED4-DOUT)
- LED7 pad 2: Net-(LED12-DIN) -> Net-(LED13-DIN)
- LED7 pad 4: Net-(LED5-DOUT) -> Net-(LED7-DIN)
- LED8 pad 2: Net-(LED13-DIN) -> Net-(LED7-DIN)
Routing:
- net +5V_{master}: track 102.6 -> 1086.4 mm, vias 1 -> 0
- net +5V: track 1697.4 -> 781.8 mm
- net LEDs^{a}: track 0.00 -> 170.2 mm, vias 0 -> 2
- net Net-(LED29-DOUT): track 76.4 -> 0.00 mm, vias 4 -> 0
- net (no net): track 231.6 -> 165.4 mm, vias 9 -> 7
- net Net-(LED26-DOUT): track 42.4 -> 0.35 mm, vias 4 -> 0
- net Net-(LED25-DOUT): track 32.9 -> 0.00 mm, vias 4 -> 0
- net Net-(LED31-DIN): track 0.00 -> 28.2 mm, vias 0 -> 2
- net Net-(LED21-DIN): track 17.3 -> 0.00 mm, vias 2 -> 0
- net Net-(LED19-DOUT): track 17.1 -> 0.00 mm, vias 2 -> 0
- net Net-(LED5-DOUT): track 41.1 -> 24.1 mm
- net Net-(LED10-DIN): track 31.8 -> 15.1 mm, vias 4 -> 2
- net COL5^{a}: track 184.1 -> 167.6 mm
- net Net-(LED27-DOUT): track 15.8 -> 0.00 mm, vias 2 -> 0
- net Net-(LED18-DOUT): track 38.0 -> 22.8 mm, vias 4 -> 2
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Other:
- board text added: "GND"
