File: pcbs/rev2.0/right.kicad_sch (KiCad schematic)
At the start: 34 parts, among them J2 Conn_ST_STDC14, SW66 MK-12C03-G015, U10 GT-TC020A-H035-L05, U6 LDI1117, U7 USBLC6-2SC6_C5261088, U8 358, U9 STM32F446RCTx, Y2 8MHz

Commit message: Finish Layout for Master Half.
- Unimplemented handedness yet.
- Rest of the board should be working already
Parts:
- removed D69: GLED, easyeda2kicad:LED0805-R-RD, symbol Device:LED
- removed D70: YLED, easyeda2kicad:LED0805-R-RD, symbol Device:LED
- removed R10: 33Ω, Resistor_SMD:R_0603_1608Metric, symbol Device:R
- removed R11: 300, Resistor_SMD:R_0603_1608Metric, symbol Device:R
- added R3: 10kΩ, Resistor_SMD:R_0805_2012Metric, symbol Device:R
Connections:
- net SWCLKb is gone; now on net SWCLK^{b}: J2.6 (JCLK/SWCLK)
- net SWDIOb is gone; now on net SWDIO^{b}: J2.4 (JTMS/SWDIO)
- net SWOb is gone; now on net SWO^{b}: J2.8 (JTDO/SWO)
- net UART_RXb is gone; now on net UART_RX^{b}: J2.13 (VCP_RX)
- net UART_TXb is gone; now on net UART_TX^{b}: J2.14 (VCP_TX)
- net USART1_TX^{b} is gone; now on net USART_TX^{b}: U9.58 (PB6)
- net +3.3V_{slave}: now also C18.2, C19.2, C20.2, C21.2, C22.2, C23.2
- net COL0^{b}: now also U9.37 (PC6); no longer U9.62 (PB9)
- net COL1^{b}: now also U9.38 (PC7); no longer U9.61 (PB8)
- net COL2^{b}: now also U9.39 (PC8); no longer U9.57 (PB5)
- net COL3^{b}: now also U9.40 (PC9); no longer U9.56 (PB4)
- net COL5^{b}: now also U9.52 (PC11); no longer U9.53 (PC12)
- net CS^{b}: now also U9.29 (PB10); no longer U9.20 (PA4)
- net DataCommand^{b}: now also U9.33 (PB12); no longer U9.25 (PC5)
- net GND: now also C24.2, U9.1 (VBAT), U9.13 (VDDA), U9.19 (VDD), U9.32 (VDD), U9.48 (VDD), U9.64 (VDD), R3.2
- net LCDReset^{b}: now also U9.34 (PB13); no longer U9.24 (PC4)
- net LEDs^{b}: now also U9.61 (PB8); no longer U9.14 (PA0)
- net ROW1^{b}: now also U9.9 (PC1); no longer U9.40 (PC9)
- net ROW2^{b}: now also U9.10 (PC2); no longer U9.39 (PC8), U9.41 (PA8)
- net ROW3^{b}: now also U9.11 (PC3); no longer U9.38 (PC7), U9.50 (PA15)
- net ROW4^{b}: now also U9.24 (PC4); no longer U9.37 (PC6)
- net ROW5^{b}: now also U9.25 (PC5); no longer U9.36 (PB15)
- net SDCS^{b}: now also U9.62 (PB9); no longer U9.26 (PB0)
- net ScreenBright^{b}: now also U9.56 (PB4); no longer U9.27 (PB1)
- net UART_RX^{b}: now also U9.15 (PA1); no longer U9.43 (PA10)
- net UART_TX^{b}: now also U9.14 (PA0); no longer U9.42 (PA9)
- net Handedness^{b}: now reaches U9.28 (PB2)
- net Handedness^{b}: now also R3.1
- net COL4^{b}: now reaches U9.51 (PC10)
- net ROW0^{b}: now reaches U9.8 (PC0)
- removed net +3.3V: C18.2, C19.2, C20.2, C21.2, C22.2, C23.2, C24.2, U9.1 (VBAT), U9.13 (VDDA), U9.19 (VDD), U9.32 (VDD), U9.48 (VDD), U9.64 (VDD)
- net BOOT0b renamed BOOT0^{b}
- net RESETb renamed RESET^{b}
- net RESET^{b}: no longer J2.12 (~{RST})
- net SW_BOOT0b renamed SW_BOOT0^{b}
- net VBUSb renamed VBUS^{b}
- new net RESET^b: J2.12 (~{RST})
Other:
- note added: "handedness circuit"
- moved on the sheet: C18, C19, C20, C21, C22, C23, C24, C27, R12, R13, R14, SW66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

Commit message: ongoing work
Connections:
- net +3.3V_{slave}: now also C24.2, U9.1 (VBAT), U9.13 (VDDA), U9.19 (VDD), U9.32 (VDD), U9.48 (VDD), U9.64 (VDD)
- net GND: no longer C24.2, U9.1 (VBAT), U9.13 (VDDA), U9.19 (VDD), U9.32 (VDD), U9.48 (VDD), U9.64 (VDD)
Changed lines of the file:
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@@
+	)
+	(junction
+		(at 78.74 97.79)
+		(diameter 0)
+		(color 0 0 0 0)
 	)
 	(junction
@@
 	)
 	(junction
+		(at 78.74 81.28)
+		(diameter 0)
+		(color 0 0 0 0)
+	)
+	(junction
 		(at 72.39 97.79)
 		(diameter 0)
@@
 	(junction
 		(at 48.26 48.26)
-		(diameter 0)
-		(color 0 0 0 0)
-	)
-	(junction
-		(at 74.93 92.71)
 		(diameter 0)
 		(color 0 0 0 0)
@@
 	(wire
 		(pts
+			(xy 78.74 97.79) (xy 78.74 81.28)
+		)
+		(stroke
+			(width 0)
+			(type default)
+		)
+	)
+	(wire
+		(pts
 			(xy 35.56 110.49) (xy 35.56 115.57)
 		)
@@
 	(wire
 		(pts
-			(xy 77.47 97.79) (xy 80.01 97.79)
+			(xy 77.47 97.79) (xy 78.74 97.79)
 		)
 		(stroke
@@
 	(wire
 		(pts
-			(xy 74.93 92.71) (xy 74.93 97.79)
-		)
-		(stroke
+			(xy 78.74 97.79) (xy 80.01 97.79)
+		)
+		(stroke
